Commit message: fix urdf

File: base_description/urdf/mecanum.urdf.xacro (robot description, xacro)
@@ -4,5 +4,5 @@
 	<include filename="$(find realsense2_description)/urdf/_d435.urdf.xacro" />
 	<!-- parameters -->
-	<xacro:arg name="rs_mount_xyz" default="0.155 0.0 0.16" />
+	<xacro:arg name="rs_mount_xyz" default="0.35 0.0 0.16" />
   	<xacro:arg name="rs_mount_rpy" default="0.0 0.0 0.0" />
 	<xacro:arg name="d400_xyz" default="0.0 0.0 0.0" />
@@ -25,5 +25,5 @@
 			<visual>
 				<geometry>
-					<cylinder radius="0.20" length="0.078" />
+					<cylinder radius="0.10" length="0.078" />
 				</geometry>
 				<material name="red"/>
@@ -41,5 +41,5 @@
 			<visual>
 				<geometry>
-					<cylinder radius="0.10" length="0.051" />
+					<cylinder radius="0.05" length="0.051" />
 				</geometry>
 				<material name="red"/>
@@ -64,5 +64,5 @@
 			<origin xyz="0 0 0" rpy="0 0 0" />
 			<geometry>
-				<box size="0.55 0.42 0.20" />
+				<box size="0.50 0.42 0.10" />
 			</geometry>
 			<material name="gray" />
